File: _autosave-keanu-homeboy.kicad_pcb (KiCad board)
At the start: 2 copper layers, 64.6 x 98.8 mm, 13 parts, among them X1 Badgelife_sao_connector_v169b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

Commit message: final keanu
Parts:
- removed the G*** at (0.00, 0.00) (x6)
- added G*** (x6): LOGO, LOGO, F.Cu at (0.00, 0.00)
Changed lines of the file:
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@@
     (visible_elements 7FFFFFFF)
     (pcbplotparams
-      (layerselection 0x010f0_80000001)
+      (layerselection 0x010f0_ffffffff)
       (usegerberextensions false)
       (usegerberattributes false)
@@
       (outputformat 1)
       (mirror false)
-      (drillshape 1)
+      (drillshape 0)
       (scaleselection 1)
       (outputdirectory "gerbers/"))
