File: keanu-homeboy.kicad_sch (KiCad schematic)
At the start: 8 parts, among them X1 Badgelife_sao_connector_v169b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

Commit message: updates for production
Parts:
- removed X1: Badgelife_sao_connector_v169bis, my-ki-cad-parts:Badgelife-SAOv169-SAO-2x3, symbol badgelife_shitty_addon_v169bis:Badgelife_sao_connector_v169bis
- added X1: Badgelife_sao_connector_v169bis, BadgePirateFootprints:Badgelife-SAOv169-SAO_Side_B.SLK, symbol BadgePiratesSymbols:Badgelife_sao_connector_v169bis
- D1, D2, D3, D4: footprint LED_SMD:LED_1206_3216Metric -> BadgePiratesFootprint:QBLP615
- R1, R2: footprint Resistor_SMD:R_1806_4516Metric -> Resistor_SMD:R_0805_2012Metric_Pad1.20x1.40mm_HandSolder
Connections:
- net GND: now also X1.2 (GND)
- net VDD: now also X1.1 (VCC)
